File: keyboard-pcb-rpi-pico-1x25.kicad_pcb (KiCad board)
At the start: 2 copper layers, 22.9 x 499.1 mm, 28 parts, among them SW1 SW_Push, SW10 SW_Push, SW11 SW_Push, SW12 SW_Push, SW13 SW_Push, SW14 SW_Push, SW15 SW_Push, SW16 SW_Push, SW17 SW_Push, SW18 SW_Push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

Commit message: Add text
Other:
- board text added: "D 3 5 G"
- board text added: "GP28 3.3V 5V GND"
- board text added: "JLCJLCJLCJLC"
- board text added: "https://github.com/nomis/keyboard-pcb-rpi-pico-1x25"
- board text added: "urn:oid:1.3.6.1.4.1.39777.1.3.2.1.0"
Changed lines of the file:
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@@
 		(layer "Edge.Cuts")
+	)
+	(gr_text "D\n3\n5\nG"
+		(at 64.77 143.51 0)
+		(layer "B.SilkS")
+		(effects
+			(font
+				(size 1.5 1.5)
+				(thickness 0.3)
+				(bold yes)
+			)
+			(justify bottom mirror)
+		)
+	)
+	(gr_text "urn:oid:1.3.6.1.4.1.39777.1.3.2.1.0"
+		(at 46.99 490.22 270)
+		(layer "B.SilkS")
+		(effects
+			(font
+				(size 1.5 1.5)
+				(thickness 0.3)
+				(bold yes)
+			)
+			(justify bottom mirror)
+		)
+	)
+	(gr_text "GP28\n3.3V\n5V\nGND"
+		(at 52.07 134.62 0)
+		(layer "B.SilkS")
+		(effects
+			(font
+				(size 1.5 1.5)
+				(thickness 0.3)
+				(bold yes)
+			)
+			(justify left top mirror)
+		)
+	)
+	(gr_text "JLCJLCJLCJLC"
+		(at 55.88 534.67 0)
+		(layer "B.SilkS")
+		(effects
+			(font
+				(size 1.5 1.5)
+				(thickness 0.3)
+				(bold yes)
+			)
+			(justify bottom mirror)
+		)
+	)
+	(gr_text "https://github.com/nomis/keyboard-pcb-rpi-pico-1x25\n\n"
+		(at 44.45 389.89 270)
+		(layer "B.SilkS")
+		(effects
+			(font
+				(size 1.5 1.5)
+				(thickness 0.3)
+				(bold yes)
+			)
+			(justify bottom mirror)
+		)
 	)
 	(dimension

Commit message: Add mounting holes and art
Parts:
- added EHLAB: LOGO, LOGO, B.Cu at (55.9, 177.4)
- added FEZ1: LOGO, LOGO, B.Cu at (47.0, 289.6)
- added FEZ2: LOGO, LOGO, B.Cu at (55.9, 158.4)
- added H1: MountingHole_Pad, MountingHole:MountingHole_3.2mm_M3_Pad, F.Cu at (55.9, 239.4)
- added H2: MountingHole_Pad, MountingHole:MountingHole_3.2mm_M3_Pad, F.Cu at (55.9, 339.7)
- added H3: MountingHole_Pad, MountingHole:MountingHole_3.2mm_M3_Pad, F.Cu at (55.9, 440.1)
- added MrMeeseeks: LOGO, LOGO, B.Cu at (55.9, 115.3)

Commit message: Move top mounting hole further up
Parts:
- moved H1 100.3 mm to (55.9, 139.1)
- moved LEDS1 100.3 mm to (63.0, 235.5)
Routing:
- net +5V: track 117.4 -> 217.7 mm
- net GP28: track 94.6 -> 194.9 mm
- net +3.3V: track 102.9 -> 203.2 mm
