File: keyboard-pcb-rpi-pico-1x25.kicad_pcb (KiCad board)
At the start: 2 copper layers, 22.9 x 499.1 mm, 35 parts, among them SW1 SW_Push, SW10 SW_Push, SW11 SW_Push, SW12 SW_Push, SW13 SW_Push, SW14 SW_Push, SW15 SW_Push, SW16 SW_Push, SW17 SW_Push, SW18 SW_Push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

Commit message: Add spider
Parts:
- added Spider: LOGO, LOGO, B.Cu at (55.9, 215.9)
Changed lines of the file:
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@@
+	(footprint "LOGO"
+		(layer "B.Cu")
+		(at 55.88 215.9 180)
+		(property "Reference" "Spider"
+			(at 0 0 0)
+			(layer "B.SilkS")
+			(hide yes)
+			(effects
+				(font
+					(size 1.5 1.5)
+					(thickness 0.3)
+				)
+				(justify mirror)
+			)
+		)
+		(property "Value" "LOGO"
+			(at 0.75 0 0)
+			(layer "B.SilkS")
+			(hide yes)
+			(effects
+				(font
+					(size 1.5 1.5)
+					(thickness 0.3)
+				)
+				(justify mirror)
+			)
+		)
+		(property "Footprint" ""
+			(at 0 0 0)
+			(layer "B.Fab")
+			(hide yes)
+			(effects
+				(font
+					(size 1.27 1.27)
+					(thickness 0.15)
+				)
+				(justify mirror)
+			)
+		)
+		(property "Datasheet" ""
+			(at 0 0 0)
+			(layer "B.Fab")
+			(hide yes)
+			(effects
+				(font
+					(size 1.27 1.27)
+					(thickness 0.15)
+				)
+				(justify mirror)
+			)
+		)
+		(property "Description" ""
+			(at 0 0 0)
+			(layer "B.Fab")
+			(hide yes)
+			(effects
+				(font
+					(size 1.27 1.27)
+					(thickness 0.15)
+				)
+				(justify mirror)
+			)
+		)
+		(attr board_only exclude_from_pos_files exclude_from_bom)
+		(fp_poly
+			(pts
+				(xy 1.573957 4.484562) (xy 2.099363 4.447661) (xy 2.231824 4.435011) (xy 2.477938 4.407794) (xy 2.643902 4.380701)
+				(xy 2.750995 4.347993) (xy 2.820499 4.303929) (xy 2.8553 4.266847) (xy 2.92045 4.120436) (xy 2.884435 3.967828)
+				(xy 2.769885 3.829774) (xy 2.724815 3.792656) (xy 2.672945 3.765785) (xy 2.599163 3.748025) (xy 2.488356 3.73824)
+				(xy 2.325414 3.735294) (xy 2.095224 3.73805) (xy 1.782676 3.745372) (xy 1.682169 3.747986) (xy 0.711958 3.773424)
+				(xy 0.641817 3.601212) (xy 0.58188 3.42324) (xy 0.539157 3.247142) (xy 0.506638 3.065284) (xy 0.930893 2.855058)
+				(xy 1.355147 2.644832) (xy 2.003978 2.973416) (xy 2.266934 3.104806) (xy 2.461874 3.195769) (xy 2.610459 3.253636)
+				(xy 2.734348 3.285737) (xy 2.855202 3.299403) (xy 2.974883 3.302) (xy 3.282371 3.268112) (xy 3.660528 3.16749)
+				(xy 4.104803 3.001702) (xy 4.610648 2.772314) (xy 4.826571 2.66445) (xy 5.098694 2.519061) (xy 5.2882 2.402194)
+				(xy 5.407194 2.30563) (xy 5.462109 2.233054) (xy 5.505178 2.055619) (xy 5.456312 1.895107) (xy 5.323936 1.776391)
+				(xy 5.304219 1.766762) (xy 5.236604 1.744118) (xy 5.162497 1.745237) (xy 5.061767 1.776533) (xy 4.914283 1.844422)
+				(xy 4.69991 1.955317) (xy 4.680899 1.965375) (xy 4.342961 2.133835) (xy 4.000082 2.286012) (xy 3.671513 2.414801)
+				(xy 3.376501 2.513101) (xy 3.134298 2.573806) (xy 2.986718 2.590552) (xy 2.774468 2.558019) (xy 2.512609 2.457697)
+				(xy 2.413 2.40903) (xy 2.18993 2.292254) (xy 2.047142 2.205783) (xy 1.972883 2.136882) (xy 1.955401 2.072816)
+				(xy 1.982942 2.00085) (xy 2.004405 1.966279) (xy 2.088444 1.838019) (xy 2.463292 2.01121) (xy 2.84046 2.145631)
+				(xy 3.190829 2.189889) (xy 3.507314 2.143565) (xy 3.658836 2.08217) (xy 3.826051 1.982939) (xy 4.046022 1.831765)
+				(xy 4.305774 1.639496) (xy 4.59233 1.416983) (xy 4.892715 1.175073) (xy 5.193954 0.924617) (xy 5.483069 0.676462)
+				(xy 5.747087 0.441457) (xy 5.97303 0.230452) (xy 6.147924 0.054296) (xy 6.258792 -0.076162) (xy 6.280501 -0.109795)
+				(xy 6.343174 -0.294948) (xy 6.308719 -0.454867) (xy 6.232425 -0.549944) (xy 6.126237 -0.630796)
+				(xy 6.020318 -0.661211) (xy 5.900628 -0.635827) (xy 5.75313 -0.54928) (xy 5.563784 -0.396206) (xy 5.371359 -0.220945)
+				(xy 4.739584 0.349407) (xy 4.143426 0.844103) (xy 3.683 1.191287) (xy 3.457476 1.343648) (xy 3.278827 1.432532)
+				(xy 3.117425 1.461322) (xy 2.943647 1.433402) (xy 2.727868 1.352157) (xy 2.635247 1.310981) (xy 2.365672 1.188656)
+				(xy 2.380521 0.759019) (xy 2.381785 0.498961) (xy 2.361022 0.297329) (xy 2.312844 0.112324) (xy 2.288191 0.042919)
+				(xy 2.102513 -0.311502) (xy 1.832638 -0.615783) (xy 1.484722 -0.866247) (xy 1.064923 -1.059215)
+				(xy 0.579398 -1.191007) (xy 0.120673 -1.252103) (xy -0.292053 -1.284008) (xy -0.354465 -1.467504)
+				(xy -0.399338 -1.666625) (xy -0.429482 -1.939806) (xy -0.444565 -2.260532) (xy -0.444255 -2.602287)
+				(xy -0.428219 -2.938557) (xy -0.396123 -3.242825) (xy -0.378127 -3.3528) (xy -0.318561 -3.683406)
+				(xy -0.280286 -3.930493) (xy -0.263382 -4.109904) (xy -0.26793 -4.237481) (xy -0.294009 -4.329066)
+				(xy -0.341701 -4.400501) (xy -0.38365 -4.443006) (xy -0.506947 -4.540917) (xy -0.602645 -4.561691)
+				(xy -0.704989 -4.508797) (xy -0.741842 -4.479306) (xy -0.823396 -4.400491) (xy -0.887517 -4.306088)
+				(xy -0.942166 -4.176128) (xy -0.995299 -3.990643) (xy -1.054877 -3.729663) (xy -1.071099 -3.653195)
+				(xy -1.138947 -3.232476) (xy -1.176307 -2.780283) (xy -1.183037 -2.32645) (xy -1.158992 -1.900814)
+				(xy -1.104029 -1.533209) (xy -1.081744 -1.439664) (xy -0.985518 -1.075928) (xy -1.165859 -0.991284)
+				(xy -1.300251 -0.920408) (xy -1.480363 -0.815409) (xy -1.667577 -0.698812) (xy -1.670441 -0.696961)
+				(xy -1.994682 -0.487282) (xy -2.317309 -0.659659) (xy -2.642821 -0.861339) (xy -2.934308 -1.094913)
+				(xy -3.16758 -1.339287) (xy -3.279298 -1.498619) (xy -3.346428 -1.627366) (xy -3.439909 -1.825772)
+				(xy -3.5485 -2.069109) (xy -3.660958 -2.332645) (xy -3.687245 -2.39608) (xy -3.793048 -2.64357)
+				(xy -3.892741 -2.859767) (xy -3.977071 -3.025786) (xy -4.036788 -3.122745) (xy -4.050201 -3.1369)
+				(xy -4.191294 -3.192433) (xy -4.353302 -3.188599) (xy -4.485079 -3.127288) (xy -4.492172 -3.120571)
+				(xy -4.552068 -3.011388) (xy -4.572 -2.89608) (xy -4.552929 -2.799084) (xy -4.500769 -2.628823)
+				(xy -4.423101 -2.405135) (xy -4.327503 -2.147862) (xy -4.221556 -1.876842) (xy -4.11284 -1.611915)
+				(xy -4.008935 -1.37292) (xy -3.917421 -1.179698) (xy -3.912658 -1.170324) (xy -3.752439 -0.930187)
+				(xy -3.515156 -0.673996) (xy -3.219517 -0.419618) (xy -2.884231 -0.184916) (xy -2.87414 -0.178606)
+				(xy -2.703251 -0.068155) (xy -2.571308 0.024623) (xy -2.497909 0.085597) (xy -2.4892 0.098985) (xy -2.523036 0.158578)
+				(xy -2.5781 0.215669) (xy -2.625383 0.24938) (xy -2.687947 0.269967) (xy -2.783076 0.277674) (xy -2.928056 0.272746)
+				(xy -3.140173 0.255428) (xy -3.420744 0.227607) (xy -3.925211 0.130899) (xy -4.442118 -0.051884)
+				(xy -4.94999 -0.311046) (xy -5.427352 -0.63689) (xy -5.54297 -0.730623) (xy -5.720415 -0.873949)
+				(xy -5.880493 -0.992985) (xy -6.000275 -1.071166) (xy -6.042015 -1.091188) (xy -6.201549 -1.094921)
+				(xy -6.365272 -1.028229) (xy -6.489594 -0.910356) (xy -6.50314 -0.887618) (xy -6.53666 -0.801284)
+				(xy -6.521814 -0.721489) (xy -6.449539 -0.610512) (xy -6.43052 -0.585348) (xy -6.212239 -0.346624)
+				(xy -5.919807 -0.096169) (xy -5.576649 0.149448) (xy -5.206194 0.373653) (xy -4.885003 0.533444)
+				(xy -0.141483 0.533444) (xy -0.094399 0.433025) (xy 0.01341 0.335836) (xy 0.163217 0.256566) (xy 0.336297 0.209903)
+				(xy 0.425076 0.20339) (xy 0.561876 0.218347) (xy 0.679133 0.276519) (xy 0.815746 0.397399) (xy 0.819281 0.400929)
+				(xy 0.947766 0.551446) (xy 0.989766 0.658519) (xy 0.98567 0.680329) (xy 0.949698 0.74309) (xy 0.896073 0.751228)
+				(xy 0.804383 0.699931) (xy 0.6858 0.6096) (xy 0.555862 0.511407) (xy 0.460958 0.469369) (xy 0.362921 0.480421)
+				(xy 0.223587 0.5415) (xy 0.169893 0.56819) (xy 0.016801 0.633512) (xy -0.075417 0.64199) (xy -0.109116 0.622405)
+				(xy -0.141483 0.533444) (xy -4.885003 0.533444) (xy -4.831869 0.559878) (xy -4.779868 0.582236)
+				(xy -4.454874 0.70005) (xy -4.07688 0.807452) (xy -3.691193 0.89322) (xy -3.343116 0.946131) (xy -3.291072 0.95104)
+				(xy -3.118997 0.967994) (xy -2.995452 0.984987) (xy -2.946447 0.998421) (xy -2.9464 0.998735) (xy -2.958932 1.05372)
+				(xy -2.991509 1.177704) (xy -3.022409 1.290548) (xy -0.077962 1.290548) (xy -0.008653 1.202089)
+				(xy 0.104349 1.178874) (xy 0.194944 1.213023) (xy 0.241363 1.291668) (xy 0.245744 1.377345) (xy 0.193282 1.476159)
+				(xy 0.1795 1.482567) (xy 0.576791 1.482567) (xy 0.587592 1.378477) (xy 0.6081 1.348007) (xy 0.711295 1.286187)
+				(xy 0.782954 1.280249) (xy 0.862136 1.319025) (xy 0.888514 1.421871) (xy 0.889 1.4478) (xy 0.874978 1.557079)
+				(xy 0.816894 1.596902) (xy 0.767536 1.6002) (xy 0.642807 1.56602) (xy 0.576791 1.482567) (xy 0.1795 1.482567)
+				(xy 0.096677 1.521076) (xy -0.005469 1.506632) (xy -0.074556 1.427358) (xy -0.076037 1.422916) (xy -0.077962 1.290548)
+				(xy -3.022409 1.290548) (xy -3.029263 1.315576) (xy -3.112126 1.613617) (xy -3.341154 1.645009)
+				(xy -3.555263 1.665245) (xy -3.801304 1.674624) (xy -4.049818 1.673588) (xy -4.271343 1.662579)
+				(xy -4.43642 1.64204) (xy -4.490132 1.627756) (xy -4.583409 1.577101) (xy -4.732996 1.479258) (xy -4.915483 1.350027)
+				(xy -5.047005 1.25184) (xy -5.281666 1.076902) (xy -5.454814 0.961254) (xy -5.58265 0.898746) (xy -5.68138 0.883225)
+				(xy -5.767204 0.908541) (xy -5.835405 0.952523) (xy -5.956668 1.068898) (xy -6.004147 1.189511)
+				(xy -5.974166 1.322739) (xy -5.863051 1.476959) (xy -5.667125 1.66055) (xy -5.449474 1.83223) (xy -5.188568 2.023981)
+				(xy -4.977059 2.16246) (xy -4.788551 2.256364) (xy -4.596651 2.31439) (xy -4.374965 2.345236) (xy -4.097098 2.357599)
+				(xy -3.84801 2.359937) (xy -3.14942 2.3622) (xy -3.071281 2.631001) (xy -2.941276 2.918731) (xy -2.738995 3.174166)
+				(xy -2.489495 3.368174) (xy -2.3961 3.415974) (xy -2.21047 3.485495) (xy -2.014348 3.529361) (xy -1.793782 3.546922)
+				(xy -1.534819 3.537528) (xy -1.223505 3.500529) (xy -0.845888 3.435275) (xy -0.388015 3.341118)
+				(xy -0.2794 3.317401) (xy -0.224013 3.318695) (xy -0.177602 3.362469) (xy -0.129241 3.466612) (xy -0.068004 3.649018)
+				(xy -0.058745 3.678714) (xy 0.011261 3.880335) (xy 0.085996 4.057892) (xy 0.150675 4.176714) (xy 0.157702 4.186203)
+				(xy 0.300706 4.312798) (xy 0.507477 4.40517) (xy 0.784371 4.464079) (xy 1.137745 4.490289)
+			)
+			(stroke
+				(width 0)
+				(type solid)
+			)
+			(fill solid)
+			(layer "B.SilkS")
+		)
+	)
 	(footprint "LOGO"
 		(layer "B.Cu")

Commit message: Add CYBER
Parts:
- added CYBER: LOGO, LOGO, B.Cu at (55.9, 258.3)
