File: keyboard-pcb-rpi-pico-25x1.kicad_pcb (KiCad board)
At the start: 2 copper layers, 25.4 x 499.1 mm, 38 parts, among them SW1 SW_Push, SW10 SW_Push, SW11 SW_Push, SW12 SW_Push, SW13 SW_Push, SW14 SW_Push, SW15 SW_Push, SW16 SW_Push, SW17 SW_Push, SW18 SW_Push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

Commit message: Fix keyboard/project name
Other:
- board text added: "https://github.com/nomis/keyboard-pcb-rpi-pico-25x1"
- board text removed: "https://github.com/nomis/keyboard-pcb-rpi-pico-1x25"
Changed lines of the file:
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@@
 		)
 		(sheetname "Root")
-		(sheetfile "keyboard-pcb-rpi-pico-1x25.kicad_sch")
+		(sheetfile "keyboard-pcb-rpi-pico-25x1.kicad_sch")
 		(attr through_hole)
 		(fp_line
@@
 		)
 		(sheetname "Root")
-		(sheetfile "keyboard-pcb-rpi-pico-1x25.kicad_sch")
+		(sheetfile "keyboard-pcb-rpi-pico-25x1.kicad_sch")
 		(attr through_hole)
 		(fp_line
@@
 		)
 		(sheetname "Root")
-		(sheetfile "keyboard-pcb-rpi-pico-1x25.kicad_sch")
+		(sheetfile "keyboard-pcb-rpi-pico-25x1.kicad_sch")
 		(attr through_hole)
 		(fp_line
@@
 		(property ki_fp_filters "MountingHole*Pad*")
 		(sheetname "Root")
-		(sheetfile "keyboard-pcb-rpi-pico-1x25.kicad_sch")
+		(sheetfile "keyboard-pcb-rpi-pico-25x1.kicad_sch")
 		(attr exclude_from_pos_files exclude_from_bom)
 		(fp_circle
@@
 		(property ki_fp_filters "MountingHole*Pad*")
 		(sheetname "Root")
-		(sheetfile "keyboard-pcb-rpi-pico-1x25.kicad_sch")
+		(sheetfile "keyboard-pcb-rpi-pico-25x1.kicad_sch")
 		(attr exclude_from_pos_files exclude_from_bom)
 		(fp_circle
@@
 		)
 		(sheetname "Root")
-		(sheetfile "keyboard-pcb-rpi-pico-1x25.kicad_sch")
+		(sheetfile "keyboard-pcb-rpi-pico-25x1.kicad_sch")
 		(attr through_hole)
 		(fp_line
@@
 		)
 		(sheetname "Root")
-		(sheetfile "keyboard-pcb-rpi-pico-1x25.kicad_sch")
+		(sheetfile "keyboard-pcb-rpi-pico-25x1.kicad_sch")
 		(attr through_hole)
 		(fp_line
@@
 		)
 		(sheetname "Root")
-		(sheetfile "keyboard-pcb-rpi-pico-1x25.kicad_sch")
+		(sheetfile "keyboard-pcb-rpi-pico-25x1.kicad_sch")
 		(attr through_hole)
 		(fp_line
@@
 		)
 		(sheetname "Root")
-		(sheetfile "keyboard-pcb-rpi-pico-1x25.kicad_sch")
+		(sheetfile "keyboard-pcb-rpi-pico-25x1.kicad_sch")
 		(attr through_hole)
 		(fp_line
@@
 		)
 		(sheetname "Root")
-		(sheetfile "keyboard-pcb-rpi-pico-1x25.kicad_sch")
+		(sheetfile "keyboard-pcb-rpi-pico-25x1.kicad_sch")
 		(attr through_hole)
 		(fp_line
@@
 		)
 		(sheetname "Root")
-		(sheetfile "keyboard-pcb-rpi-pico-1x25.kicad_sch")
+		(sheetfile "keyboard-pcb-rpi-pico-25x1.kicad_sch")
 		(attr through_hole)
 		(fp_line
@@
 		(property ki_fp_filters "MountingHole*Pad*")
 		(sheetname "Root")
-		(sheetfile "keyboard-pcb-rpi-pico-1x25.kicad_sch")
+		(sheetfile "keyboard-pcb-rpi-pico-25x1.kicad_sch")
 		(attr exclude_from_pos_files exclude_from_bom)
 		(fp_circle
@@
 		)
 		(sheetname "Root")
-		(sheetfile "keyboard-pcb-rpi-pico-1x25.kicad_sch")
+		(sheetfile "keyboard-pcb-rpi-pico-25x1.kicad_sch")
 		(attr through_hole)
 		(fp_line
@@
 		)
 		(sheetname "Root")
-		(sheetfile "keyboard-pcb-rpi-pico-1x25.kicad_sch")
+		(sheetfile "keyboard-pcb-rpi-pico-25x1.kicad_sch")
 		(attr through_hole)
 		(fp_line
@@
 		)
 		(sheetname "Root")
-		(sheetfile "keyboard-pcb-rpi-pico-1x25.kicad_sch")
+		(sheetfile "keyboard-pcb-rpi-pico-25x1.kicad_sch")
 		(attr through_hole)
 		(fp_line
@@
 		)
 		(sheetname "Root")
-		(sheetfile "keyboard-pcb-rpi-pico-1x25.kicad_sch")
+		(sheetfile "keyboard-pcb-rpi-pico-25x1.kicad_sch")
 		(attr through_hole)
 		(fp_line
@@
 		)
 		(sheetname "Root")
-		(sheetfile "keyboard-pcb-rpi-pico-1x25.kicad_sch")
+		(sheetfile "keyboard-pcb-rpi-pico-25x1.kicad_sch")
 		(attr through_hole)
 		(fp_line
@@
 		)
 		(sheetname "Root")
-		(sheetfile "keyboard-pcb-rpi-pico-1x25.kicad_sch")
+		(sheetfile "keyboard-pcb-rpi-pico-25x1.kicad_sch")
 		(attr through_hole)
 		(fp_line
@@
 		)
 		(sheetname "Root")
-		(sheetfile "keyboard-pcb-rpi-pico-1x25.kicad_sch")
+		(sheetfile "keyboard-pcb-rpi-pico-25x1.kicad_sch")
 		(attr through_hole)
 		(fp_line
@@
 		)
 		(sheetname "Root")
-		(sheetfile "keyboard-pcb-rpi-pico-1x25.kicad_sch")
+		(sheetfile "keyboard-pcb-rpi-pico-25x1.kicad_sch")
 		(attr through_hole)
 		(fp_line
@@
 		)
 		(sheetname "Root")
-		(sheetfile "keyboard-pcb-rpi-pico-1x25.kicad_sch")
+		(sheetfile "keyboard-pcb-rpi-pico-25x1.kicad_sch")
 		(attr through_hole)
 		(fp_line
@@
 		)
 		(sheetname "Root")
-		(sheetfile "keyboard-pcb-rpi-pico-1x25.kicad_sch")
+		(sheetfile "keyboard-pcb-rpi-pico-25x1.kicad_sch")
 		(attr through_hole)
 		(fp_line
@@
 		)
 		(sheetname "Root")
-		(sheetfile "keyboard-pcb-rpi-pico-1x25.kicad_sch")
+		(sheetfile "keyboard-pcb-rpi-pico-25x1.kicad_sch")
 		(attr through_hole)
 		(fp_line
@@
 		)
 		(sheetname "Root")
-		(sheetfile "keyboard-pcb-rpi-pico-1x25.kicad_sch")
+		(sheetfile "keyboard-pcb-rpi-pico-25x1.kicad_sch")
 		(attr through_hole)
 		(fp_line
@@
 		)
 		(sheetname "Root")
-		(sheetfile "keyboard-pcb-rpi-pico-1x25.kicad_sch")
+		(sheetfile "keyboard-pcb-rpi-pico-25x1.kicad_sch")
 		(attr through_hole)
 		(fp_line
@@
 		)
 		(sheetname "Root")
-		(sheetfile "keyboard-pcb-rpi-pico-1x25.kicad_sch")
+		(sheetfile "keyboard-pcb-rpi-pico-25x1.kicad_sch")
 		(attr through_hole)
 		(fp_line
@@
 		)
 		(sheetname "Root")
-		(sheetfile "keyboard-pcb-rpi-pico-1x25.kicad_sch")
+		(sheetfile "keyboard-pcb-rpi-pico-25x1.kicad_sch")
 		(attr through_hole)
 		(fp_line
@@
 		)
 		(sheetname "Root")
-		(sheetfile "keyboard-pcb-rpi-pico-1x25.kicad_sch")
+		(sheetfile "keyboard-pcb-rpi-pico-25x1.kicad_sch")
 		(attr through_hole)
 		(fp_line
@@
 		(property ki_fp_filters "Connector*:*_1x??_*")
 		(sheetname "Root")
-		(sheetfile "keyboard-pcb-rpi-pico-1x25.kicad_sch")
+		(sheetfile "keyboard-pcb-rpi-pico-25x1.kicad_sch")
 		(attr through_hole)
 		(fp_line
@@
 		(property ki_fp_filters "Connector*:*_1x??_*")
 		(sheetname "Root")
-		(sheetfile "keyboard-pcb-rpi-pico-1x25.kicad_sch")
+		(sheetfile "keyboard-pcb-rpi-pico-25x1.kicad_sch")
 		(attr through_hole)
 		(fp_line
@@
 		(property ki_fp_filters "Connector*:*_1x??_*")
 		(sheetname "Root")
-		(sheetfile "keyboard-pcb-rpi-pico-1x25.kicad_sch")
+		(sheetfile "keyboard-pcb-rpi-pico-25x1.kicad_sch")
 		(attr through_hole)
 		(fp_line
@@
 		)
 	)
-	(gr_text "https://github.com/nomis/keyboard-pcb-rpi-pico-1x25"
+	(gr_text "https://github.com/nomis/keyboard-pcb-rpi-pico-25x1"
 		(at 46.99 389.89 270)
 		(layer "B.SilkS")
