File: keyboard-pcb-rpi-pico-25x1.kicad_pcb (KiCad board)
At the start: 2 copper layers, 25.4 x 499.1 mm, 38 parts, among them SW1 SW_Push, SW10 SW_Push, SW11 SW_Push, SW12 SW_Push, SW13 SW_Push, SW14 SW_Push, SW15 SW_Push, SW16 SW_Push, SW17 SW_Push, SW18 SW_Push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

Commit message: Move the ground to the other side of the switch pins
Connections:
- SW1 pad 1: GND -> GP0
- SW1 pad 2: GP0 -> GND
- SW10 pad 1: GND -> GP5
- SW10 pad 2: GP5 -> GND
- SW11 pad 1: GND -> GP4
- SW11 pad 2: GP4 -> GND
- SW12 pad 1: GND -> GP3
- SW12 pad 2: GP3 -> GND
- SW13 pad 1: GND -> GP15
- SW13 pad 2: GP15 -> GND
- SW14 pad 1: GND -> GP14
- SW14 pad 2: GP14 -> GND
- SW15 pad 1: GND -> GP13
- SW15 pad 2: GP13 -> GND
- SW16 pad 1: GND -> GP12
- SW16 pad 2: GP12 -> GND
- SW17 pad 1: GND -> GP19
- SW17 pad 2: GP19 -> GND
- SW18 pad 1: GND -> GP18
- SW18 pad 2: GP18 -> GND
- SW19 pad 1: GND -> GP17
- SW19 pad 2: GP17 -> GND
- SW2 pad 1: GND -> GP1
- SW2 pad 2: GP1 -> GND
- SW20 pad 1: GND -> GP16
- SW20 pad 2: GP16 -> GND
- SW21 pad 1: GND -> GP20
- SW21 pad 2: GP20 -> GND
- SW22 pad 1: GND -> GP21
- SW22 pad 2: GP21 -> GND
- SW23 pad 1: GND -> GP22
- SW23 pad 2: GP22 -> GND
- SW24 pad 1: GND -> GP26
- SW24 pad 2: GP26 -> GND
- SW25 pad 1: GND -> GP27
- SW25 pad 2: GP27 -> GND
- SW3 pad 1: GND -> GP2
- SW3 pad 2: GP2 -> GND
- SW4 pad 1: GND -> GP11
- SW4 pad 2: GP11 -> GND
- SW5 pad 1: GND -> GP10
- SW5 pad 2: GP10 -> GND
- SW6 pad 1: GND -> GP9
- SW6 pad 2: GP9 -> GND
- SW7 pad 1: GND -> GP8
- SW7 pad 2: GP8 -> GND
- SW8 pad 1: GND -> GP7
- SW8 pad 2: GP7 -> GND
- SW9 pad 1: GND -> GP6
- SW9 pad 2: GP6 -> GND
Routing:
- net GP27: track 499.0 -> 477.9 mm
- net GP1: track 36.0 -> 22.2 mm
- net GP0: track 19.0 -> 7.93 mm
- net GP11: track 34.4 -> 28.8 mm
- net GP4: track 207.3 -> 212.6 mm
- net GP26: track 462.0 -> 456.8 mm
- net GP21: track 409.4 -> 404.2 mm
- net GP12: track 276.4 -> 271.2 mm
- net GP14: track 224.8 -> 219.6 mm
- net GP13: track 249.3 -> 244.1 mm
- net GP15: track 202.1 -> 196.9 mm
- net GP22: track 435.4 -> 430.3 mm
- net GP20: track 397.7 -> 392.5 mm
- net GP2: track 43.0 -> 38.8 mm
- net GP9: track 88.8 -> 91.1 mm
Other:
- board text added: "urn:oid:1.3.6.1.4.1.39777.1.3.2.1.4"
- board text removed: "urn:oid:1.3.6.1.4.1.39777.1.3.2.1.3"

Commit message: Fix schematic power error messages by adding PWR_FLAG
Connections:
- net 3V3_EN renamed /3V3_EN
- net ADC_GND renamed /ADC_GND
- net ADC_VREF renamed /ADC_VREF
- net RUN renamed /RUN
- net VSYS renamed /VSYS
Changed lines of the file:
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@@
 	(net 28 "+5V")
 	(net 29 "+3.3V")
-	(net 30 "ADC_GND")
-	(net 31 "RUN")
-	(net 32 "3V3_EN")
-	(net 33 "VSYS")
-	(net 34 "ADC_VREF")
+	(net 30 "/ADC_GND")
+	(net 31 "/RUN")
+	(net 32 "/3V3_EN")
+	(net 33 "/VSYS")
+	(net 34 "/ADC_VREF")
 	(footprint "Button_Switch_Keyboard:SW_Cherry_MX_1.00u_PCB"
 		(layer "F.Cu")
@@
 			)
 			(remove_unused_layers no)
-			(net 33 "VSYS")
+			(net 33 "/VSYS")
 			(pinfunction "Pin_2")
-			(pintype "passive")
+			(pintype "passive+no_connect")
 		)
 		(pad "3" thru_hole oval
@@
 			)
 			(remove_unused_layers no)
-			(net 32 "3V3_EN")
+			(net 32 "/3V3_EN")
 			(pinfunction "Pin_4")
-			(pintype "passive")
+			(pintype "passive+no_connect")
 		)
 		(pad "5" thru_hole oval
@@
 			)
 			(remove_unused_layers no)
-			(net 34 "ADC_VREF")
+			(net 34 "/ADC_VREF")
 			(pinfunction "Pin_6")
-			(pintype "passive")
+			(pintype "passive+no_connect")
 		)
 		(pad "7" thru_hole oval
@@
 			)
 			(remove_unused_layers no)
-			(net 30 "ADC_GND")
+			(net 30 "/ADC_GND")
 			(pinfunction "Pin_8")
-			(pintype "passive")
+			(pintype "passive+no_connect")
 		)
 		(pad "9" thru_hole oval
@@
 			)
 			(remove_unused_layers no)
-			(net 31 "RUN")
+			(net 31 "/RUN")
 			(pinfunction "Pin_11")
-			(pintype "passive")
+			(pintype "passive+no_connect")
 		)
 		(pad "12" thru_hole oval
